Commit message: Feat: Add Rotation

File: src/cnuchacha_description/urdf/cnuchacha_macro.xacro (robot description, xacro)
@@ -22,5 +22,5 @@
         <origin xyz="0 0 ${body_h/2 + leg_l}" rpy="0 0 0"/>
         <geometry><box size="${body_d} ${body_w} ${body_h}"/></geometry>
-        <material name="navy"/>
+        <material name="black"/>
       </visual>
       <collision>
@@ -34,4 +34,25 @@
       </inertial>
     </link>
+    <!-- Hat Brim -->
+    <joint name="${prefix}hat_brim_joint" type="fixed">
+      <parent link="${prefix}base_link"/>
+      <child link="${prefix}hat_brim_link"/>
+      <origin xyz="0 0 ${leg_l + body_h + head_r}" rpy="0 0 0"/>
+    </joint>
+    <link name="${prefix}hat_brim_link">
+      <visual>
+        <origin xyz="0 0 0" rpy="0 0 0"/>
+        <geometry><box size="0.35 0.25 0.1"/></geometry>
+        <material name="blue"/>
+      </visual>
+      <collision>
+        <origin xyz="0 0 0" rpy="0 0 0"/>
+        <geometry><box size="0.35 0.25 0.1"/></geometry>
+      </collision>
+      <inertial>
+        <mass value="0.05"/>
+        <inertia ixx="0.001" ixy="0.0" ixz="0.0" iyy="0.001" iyz="0.0" izz="0.001"/>
+      </inertial>
+    </link>
     <!-- Chacha Head -->
     <joint name="${prefix}head_joint" type="fixed">
@@ -48,6 +69,11 @@
       <visual> <!-- Snout -->
         <origin xyz="${head_r*0.7} 0 0" rpy="0 ${pi/2} 0"/>
-        <geometry><cylinder radius="0.1" length="0.2"/></geometry>
-        <material name="white"/>
+        <geometry><cylinder radius="0.12" length="0.4"/></geometry>
+        <material name="beige"/>
+      </visual>
+      <visual>
+        <origin xyz="${head_r*0.7 + 0.2} 0 0" rpy="0 0 0"/>
+        <geometry><sphere radius="0.12"/></geometry>
+        <material name="beige"/>
       </visual>
       <collision>
@@ -102,4 +128,38 @@
         <mass value="${mass}"/>
         <inertia ixx="0.01" ixy="0.0" ixz="0.0" iyy="0.01" iyz="0.0" izz="0.01"/>
+      </inertial>
+    </link>
+    <!-- Left Foot -->
+    <joint name="${prefix}left_foot_joint" type="fixed">
+      <parent link="${prefix}left_leg"/>
+      <child link="${prefix}left_foot"/>
+      <origin xyz="0 0 ${-leg_l}" rpy="0 0 0"/>
+    </joint>
+    <link name="${prefix}left_foot">
+      <visual>
+        <origin xyz="0 0 0" rpy="0 0 0"/>
+        <geometry><sphere radius="0.08"/></geometry>
+        <material name="blue"/>
+      </visual>
+      <inertial>
+        <mass value="0.1"/>
+        <inertia ixx="0.001" ixy="0.0" ixz="0.0" iyy="0.001" iyz="0.0" izz="0.001"/>
+      </inertial>
+    </link>
+    <!-- Right Foot -->
+    <joint name="${prefix}right_foot_joint" type="fixed">
+      <parent link="${prefix}right_leg"/>
+      <child link="${prefix}right_foot"/>
+      <origin xyz="0 0 ${-leg_l}" rpy="0 0 0"/>
+    </joint>
+    <link name="${prefix}right_foot">
+      <visual>
+        <origin xyz="0 0 0" rpy="0 0 0"/>
+        <geometry><sphere radius="0.08"/></geometry>
+        <material name="blue"/>
+      </visual>
+      <inertial>
+        <mass value="0.1"/>
+        <inertia ixx="0.001" ixy="0.0" ixz="0.0" iyy="0.001" iyz="0.0" izz="0.001"/>
       </inertial>
     </link>
@@ -155,41 +215,78 @@
       </inertial>
     </link>
+    <!-- Left Hand -->
+    <joint name="${prefix}left_hand_joint" type="fixed">
+      <parent link="${prefix}left_arm"/>
+      <child link="${prefix}left_hand"/>
+      <origin xyz="0 0 ${-arm_l}" rpy="0 0 0"/>
+    </joint>
+    <link name="${prefix}left_hand">
+      <visual>
+        <origin xyz="0 0 0" rpy="0 0 0"/>
+        <geometry><sphere radius="0.07"/></geometry>
+        <material name="white"/>
+      </visual>
+      <inertial>
+        <mass value="0.1"/>
+        <inertia ixx="0.001" ixy="0.0" ixz="0.0" iyy="0.001" iyz="0.0" izz="0.001"/>
+      </inertial>
+    </link>
+    <!-- Right Hand -->
+    <joint name="${prefix}right_hand_joint" type="fixed">
+      <parent link="${prefix}right_arm"/>
+      <child link="${prefix}right_hand"/>
+      <origin xyz="0 0 ${-arm_l}" rpy="0 0 0"/>
+    </joint>
+    <link name="${prefix}right_hand">
+      <visual>
+        <origin xyz="0 0 0" rpy="0 0 0"/>
+        <geometry><sphere radius="0.07"/></geometry>
+        <material name="white"/>
+      </visual>
+      <inertial>
+        <mass value="0.1"/>
+        <inertia ixx="0.001" ixy="0.0" ixz="0.0" iyy="0.001" iyz="0.0" izz="0.001"/>
+      </inertial>
+    </link>
     <!-- Nupjuki (KAIST Mascot on Hat) -->
-    <joint name="${prefix}nupjuki_joint" type="fixed">
+    <joint name="${prefix}nupjuki_joint" type="revolute">
       <parent link="${prefix}head_link"/>
       <child link="${prefix}nupjuki_link"/>
       <origin xyz="0 0 ${head_r}" rpy="0 0 0"/>
+      <axis xyz="0 0 1"/>
+      <dynamics damping="0.7"/>
+      <limit effort="100" velocity="1.0" lower="-3.14" upper="3.14"/>
     </joint>
     <link name="${prefix}nupjuki_link">
       <!-- Nupjuki Body -->
       <visual>
-        <origin xyz="0 0 0.05" rpy="0 0 0"/>
-        <geometry><cylinder radius="0.04" length="0.1"/></geometry>
+        <origin xyz="0 0 0.075" rpy="0 0 0"/>
+        <geometry><cylinder radius="0.06" length="0.15"/></geometry>
         <material name="cyan"/>
       </visual>
       <!-- Nupjuki Flat Head -->
       <visual>
-        <origin xyz="0 0 0.1" rpy="0 0 0"/>
-        <geometry><box size="0.1 0.4 0.05"/></geometry>
+        <origin xyz="0 0 0.15" rpy="0 0 0"/>
+        <geometry><box size="0.15 0.6 0.075"/></geometry>
         <material name="blue"/>
       </visual>
       <!-- Left Eye -->
       <visual>
-        <origin xyz="0.05 0.08 0.1" rpy="0 ${pi/2} 0"/>
-        <geometry><cylinder radius="0.02" length="0.01"/></geometry>
+        <origin xyz="0.075 0.12 0.15" rpy="0 ${pi/2} 0"/>
+        <geometry><cylinder radius="0.03" length="0.015"/></geometry>
         <material name="black"/>
       </visual>
       <!-- Right Eye -->
       <visual>
-        <origin xyz="0.05 -0.08 0.1" rpy="0 ${pi/2} 0"/>
-        <geometry><cylinder radius="0.02" length="0.01"/></geometry>
+        <origin xyz="0.075 -0.12 0.15" rpy="0 ${pi/2} 0"/>
+        <geometry><cylinder radius="0.03" length="0.015"/></geometry>
         <material name="black"/>
       </visual>
       <collision>
-        <origin xyz="0 0 0.1" rpy="0 0 0"/>
-        <geometry><box size="0.1 0.4 0.05"/></geometry>
-      </collision>
-      <inertial>
-        <origin xyz="0 0 0.1" rpy="0 0 0"/>
+        <origin xyz="0 0 0.15" rpy="0 0 0"/>
+        <geometry><box size="0.15 0.6 0.075"/></geometry>
+      </collision>
+      <inertial>
+        <origin xyz="0 0 0.15" rpy="0 0 0"/>
         <mass value="0.1"/>
         <inertia ixx="0.001" ixy="0.0" ixz="0.0" iyy="0.001" iyz="0.0" izz="0.001"/>

File: src/cnuchacha_description/urdf/cnuchacha_materials.xacro (robot description, xacro)
@@ -16,4 +16,7 @@
   <material name="grey">
     <color rgba="0.2 0.2 0.2 1.0"/>
+  </material>
+  <material name="beige">
+    <color rgba="0.96 0.87 0.70 1.0"/>
   </material>
   <material name="orange">

File: src/cnuchacha_launcher/urdf/cnuchacha_gazebo.xacro (robot description, xacro)
@@ -10,9 +10,13 @@
     <!-- Torso -->
     <gazebo reference="${prefix}base_link">
-      <material>Gazebo/Blue</material>
+      <material>Gazebo/Black</material>
     </gazebo>
     <!-- Head -->
     <gazebo reference="${prefix}head_link">
       <material>Gazebo/White</material>
+    </gazebo>
+    <!-- Hat Brim -->
+    <gazebo reference="${prefix}hat_brim_link">
+      <material>Gazebo/Blue</material>
     </gazebo>
     <!-- Legs -->
@@ -22,4 +26,10 @@
     <gazebo reference="${prefix}right_leg">
       <material>Gazebo/White</material>
+    </gazebo>
+    <gazebo reference="${prefix}left_foot">
+      <material>Gazebo/Blue</material>
+    </gazebo>
+    <gazebo reference="${prefix}right_foot">
+      <material>Gazebo/Blue</material>
     </gazebo>
     <!-- Arms -->
@@ -36,5 +46,11 @@
     <!-- Nupjuki -->
     <gazebo reference="${prefix}nupjuki_link">
-      <material>Gazebo/SkyBlue</material>
+      <visual>
+        <material>
+          <ambient>0 1 1 1</ambient>
+          <diffuse>0 1 1 1</diffuse>
+          <specular>0 0.1 0.1 1</specular>
+        </material>
+      </visual>
     </gazebo>
   </xacro:macro>

File: src/cnuchacha_launcher/urdf/cnuchacha_ros2_control.xacro (robot description, xacro)
@@ -20,4 +20,11 @@
         <state_interface name="position"/>
       </joint>
+      <joint name="${prefix}nupjuki_joint">
+        <command_interface name="position">
+          <param name="min">-3.14</param>
+          <param name="max">3.14</param>
+        </command_interface>
+        <state_interface name="position"/>
+      </joint>
     </ros2_control>
   </xacro:macro>

Commit message: Feat: Leg folding

File: src/cnuchacha_description/urdf/cnuchacha_macro.xacro (robot description, xacro)
@@ -88,8 +88,11 @@
     </link>
     <!-- Legs -->
-    <joint name="${prefix}left_leg_joint" type="fixed">
+    <joint name="${prefix}left_leg_joint" type="revolute">
       <parent link="${prefix}base_link"/>
       <child link="${prefix}left_leg"/>
       <origin xyz="0 ${body_w/4} ${leg_l}" rpy="0 0 0"/>
+      <axis xyz="0 -1 0"/>
+      <dynamics damping="0.7"/>
+      <limit effort="100" velocity="1.0" lower="-1.57" upper="1.57"/>
     </joint>
     <link name="${prefix}left_leg">
@@ -109,8 +112,11 @@
       </inertial>
     </link>
-    <joint name="${prefix}right_leg_joint" type="fixed">
+    <joint name="${prefix}right_leg_joint" type="revolute">
       <parent link="${prefix}base_link"/>
       <child link="${prefix}right_leg"/>
       <origin xyz="0 ${-body_w/4} ${leg_l}" rpy="0 0 0"/>
+      <axis xyz="0 -1 0"/>
+      <dynamics damping="0.7"/>
+      <limit effort="100" velocity="1.0" lower="-1.57" upper="1.57"/>
     </joint>
     <link name="${prefix}right_leg">

File: src/cnuchacha_launcher/urdf/cnuchacha_ros2_control.xacro (robot description, xacro)
@@ -27,4 +27,18 @@
         <state_interface name="position"/>
       </joint>
+      <joint name="${prefix}left_leg_joint">
+        <command_interface name="position">
+          <param name="min">-1.57</param>
+          <param name="max">1.57</param>
+        </command_interface>
+        <state_interface name="position"/>
+      </joint>
+      <joint name="${prefix}right_leg_joint">
+        <command_interface name="position">
+          <param name="min">-1.57</param>
+          <param name="max">1.57</param>
+        </command_interface>
+        <state_interface name="position"/>
+      </joint>
     </ros2_control>
   </xacro:macro>
